File: Diseños_PCB/MainBoard_ESP8266/MainBoard_ESP8266.kicad_pcb (KiCad board)
At the start: 2 copper layers, 34 parts, among them J1 Input_BAT, J2 USB_B_Micro, J3 FTDI, Q1 2N7002, SW2 SW_Push, SW3 SW_Push, U2 AMS1117-3.3, U3 ESP-12F, U4 MT3608

Commit message: Actualizacion PCB
Parts:
- added R9: 2,2K, Resistor_SMD:R_0805_2012Metric_Pad1.20x1.40mm_HandSolder, B.Cu at (169.5, 124.5)
- added SW1: SW_SPDT, EESTN5-v2:SW_SPDT_TH_100Mils_VERTICAL, F.Cu at (151.8, 115.0)
- added U5: TP4056, TP4056:SOP127P600X175-9N, B.Cu at (140.3, 120.0)
- C1, C2, C3, C4, C6, C7, D1, D2, D3, J1, J2, L1, R1, R2, R3, U2, U4: moved to B.Cu
- RV1: footprint Potentiometer_THT:Potentiometer_Vishay_T73YP_Vertical -> Potentiometer_THT:Potentiometer_Bourns_3266P_Horizontal; moved to B.Cu
- moved R11 87.8 mm to (144.1, 70.5), turned to 90 degrees
- moved R10 87.3 mm to (140.8, 70.5), turned to 90 degrees
- moved D4 86.5 mm to (135.2, 70.9), turned to 90 degrees
- moved D5 78.4 mm to (142.7, 77.0), turned to 90 degrees
- moved Q1 67.9 mm to (142.2, 84.4), turned to 90 degrees
- moved RV1 64.7 mm to (177.7, 122.1), turned to 90 degrees
- moved BZ1 63.9 mm to (133.6, 86.9), turned to 90 degrees
- moved C7 62.2 mm to (167.9, 120.0), turned to 180 degrees
- moved R12 57.8 mm to (142.0, 91.6), turned to 90 degrees
- moved C6 56.8 mm to (163.6, 124.9)
- moved L1 51.8 mm to (160.6, 116.1)
- moved D3 49.7 mm to (171.6, 116.1), turned to 180 degrees
- moved C3 49.0 mm to (179.6, 109.9), turned to -90 degrees
- moved C1 42.9 mm to (144.5, 123.9)
- moved U4 42.7 mm to (162.4, 121.7), turned to 180 degrees
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Routing:
- net GND: track 0.00 -> 97.3 mm, vias 0 -> 2
- net Net-(D1-A): track 0.00 -> 45.9 mm
- net /VB: track 0.00 -> 35.0 mm
- net Net-(SW1-A): track 0.00 -> 21.2 mm
- net +5V: track 0.00 -> 21.0 mm
- net Net-(U4-FB): track 0.00 -> 16.8 mm
- net +3.3V: track 0.00 -> 15.2 mm
- net unconnected-(J2-Shield-Pad6): track 0.00 -> 12.6 mm
- net Net-(D3-A2): track 0.00 -> 10.3 mm
- net Net-(R9-Pad1): track 0.00 -> 8.21 mm
- net Net-(U5-~{CHRG}): track 0.00 -> 6.31 mm
- net Net-(U5-~{STDBY}): track 0.00 -> 6.17 mm
- net Net-(U5-PROG): track 0.00 -> 5.06 mm
- net Net-(D2-K): track 0.00 -> 2.08 mm
- net Net-(D1-K): track 0.00 -> 2.07 mm
Other:
- board outline added: 60 x 60 mm

Commit message: Edicion archivos pcb
Parts:
- removed J3: FTDI, Connector_PinHeader_2.54mm:PinHeader_1x04_P2.54mm_Horizontal
- added J4: Sensor, Connector_PinHeader_2.54mm:PinHeader_1x03_P2.54mm_Horizontal, B.Cu at (155.3, 106.6)
- added J5: FTDI, Connector_PinHeader_2.54mm:PinHeader_1x03_P2.54mm_Horizontal, B.Cu at (133.8, 104.1)
- C5, Q1, R10, R11, R12, R4, R5, R6, R7, SW1, SW2, SW3, U3: moved to B.Cu
- moved SW3 43.8 mm to (139.5, 97.5), turned to 180 degrees
- moved SW2 42.9 mm to (139.5, 90.2)
- moved R12 25.8 mm to (159.9, 73.1), turned to 180 degrees
- moved C5 21.8 mm to (173.0, 104.1)
- moved D5 20.6 mm to (124.3, 86.2)
- moved R11 19.9 mm to (131.8, 86.2), turned to 180 degrees
- moved R5 18.6 mm to (167.4, 74.4), turned to -90 degrees
- moved R7 18.5 mm to (168.1, 103.8)
- moved R6 17.1 mm to (173.1, 74.4), turned to -90 degrees
- moved R4 14.4 mm to (170.2, 74.4), turned to -90 degrees
- moved U3 13.8 mm to (158.8, 92.8), turned to -90 degrees
- moved D4 13.7 mm to (124.3, 79.1)
- moved BZ1 13.6 mm to (142.5, 76.7), turned to 180 degrees
- moved R10 12.4 mm to (131.8, 79.1), turned to 180 degrees
- moved Q1 12.1 mm to (148.3, 74.0), turned to 180 degrees
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Connections:
- U3 pad 19: unconnected-(U3-GPIO4-Pad19) -> /PIR
- U3 pad 5: /BUZZER -> /LED_WIFI
- U3 pad 7: /LED_WIFI -> /BUZZER
Routing:
- net GND: track 97.3 -> 288.9 mm, vias 2 -> 6
- net +5V: track 21.0 -> 128.5 mm
- net Net-(U3-GPIO0): track 0.00 -> 72.4 mm, vias 0 -> 3
- net +3.3V: track 15.2 -> 67.8 mm
- net Net-(U3-~{RST}): track 0.00 -> 40.3 mm, vias 0 -> 2
- net /LED_STATUS: track 0.00 -> 38.5 mm
- net /LED_WIFI: track 0.00 -> 37.6 mm
- net /Rx: track 0.00 -> 27.7 mm
- net /Tx: track 0.00 -> 24.0 mm
- net Net-(U3-EN): track 0.00 -> 22.9 mm, vias 0 -> 2
- net /BUZZER: track 0.00 -> 16.0 mm
- net /PIR: track 0.00 -> 12.0 mm
- net Net-(Q1-G): track 0.00 -> 9.11 mm
- net Net-(D5-A): track 0.00 -> 4.76 mm
- net Net-(D4-A): track 0.00 -> 4.76 mm
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- added copper zone on B.Cu, net /VB
- added copper zone on F.Cu, net /VB
- added copper zone on B.Cu, net GND
- added copper zone on F.Cu, net GND
Other:
- board size 60 x 60 mm -> 57 x 60 mm

Commit message: Mejoras PCB
Parts:
- added H1: Hole, EESTN5-v2:Separador_M3_5mm, F.Cu at (126.2, 95.0)
- RV1: moved to F.Cu
- moved RV1 5.05 mm to (166.0, 125.5)
- moved C6 3.84 mm to (153.0, 128.5), turned to 180 degrees
Routing:
- net Net-(SW1-A): track 21.2 -> 16.7 mm
- net Net-(R9-Pad1): track 8.21 -> 4.14 mm
- net GND: track 288.9 -> 292.7 mm, vias 6 -> 7
- net +5V: track 128.5 -> 131.5 mm
- net Net-(U4-FB): track 16.8 -> 15.7 mm
