File: Diseños_PCB/MainBoard_ESP8266/MainBoard_ESP8266.kicad_sch (KiCad schematic)
At the start: 26 parts, among them J1 Input_BAT, J2 USB_B_Micro, J3 FTDI, SW1 SW_SPST, SW2 SW_Push, SW3 SW_Push, SW4 SW_Push_Dual, SW5 SW_Push_Dual, SW6 SW_Push_Dual, U1 TP4056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

Commit message: Diseño del esquematico terminado
Parts:
- removed SW1: SW_SPST, Button_Switch_SMD:SW_SPDT_PCM12, symbol Switch:SW_SPST
- removed SW4, SW5, SW6: SW_Push_Dual, Button_Switch_SMD:SW_SPST_TL3342, symbol Switch:SW_Push_Dual
- added BZ1: Buzzer, EESTN5-v2:Buzzer_12mm, symbol Device:Buzzer
- added C2 (x2): 22uF, Capacitor_SMD:C_1206_3216Metric_Pad1.33x1.80mm_HandSolder, symbol Device:C
- added D3: SS34, Diode_SMD:D_SMB_Handsoldering, symbol Diode:SM6T6V8A
- added D4: LED, EESTN5-v2:led_5mm_red, symbol Device:LED
- added D5: LED, EESTN5-v2:led_5mm_green, symbol Device:LED
- added L1: 22uH, Inductor_SMD:L_6.3x6.3_H3, symbol Device:L
- added Q1: 2N7002, Package_TO_SOT_SMD:SOT-23, symbol Transistor_FET:2N7002
- added R6 (x2): 220, Resistor_SMD:R_1206_3216Metric_Pad1.30x1.75mm_HandSolder, symbol Device:R
- added R6: 10K, Resistor_SMD:R_1206_3216Metric_Pad1.30x1.75mm_HandSolder, symbol Device:R
- added R9: 2,2K, symbol Device:R
- added RV1: 100K, Potentiometer_THT:Potentiometer_Vishay_T73YP_Vertical, symbol Device:R_Potentiometer
- added SW1: SW_SPDT, symbol Switch:SW_SPDT
- added U4: MT3608, Package_TO_SOT_SMD:SOT-23-6, symbol Regulator_Switching:MT3608
Connections:
- net GND: now also C2.2, C2.2, D4.1 (K), D5.1 (K), Q1.2 (S), R9.2, U4.2 (GND)
- net LED_WIFI: now reaches U3.7 (GPIO13)
- net LED_WIFI: now also R6.1
- net LED_STATUS: now reaches U3.6 (GPIO12)
- net LED_STATUS: now also R6.1
- net BUZZER: now reaches U3.5 (GPIO14)
- net BUZZER: now also R6.1
- net VBAT renamed VB
- net VB: now also SW1.2 (B)
- net VCC_OLED renamed +5V
- net +5V: now also BZ1.1 (-), C2.1, D3.1 (A1), RV1.3
- new net: D5.2 (A), R6.2
- new net: D3.2 (A2), L1.2, U4.1 (SW)
- new net: R9.1, RV1.1
- new net: RV1.2, U4.3 (FB)
- new net: C2.1, L1.1, SW1.1 (A), U4.4 (EN), U4.5 (IN)
- new net: D4.2 (A), R6.2
- new net: Q1.1 (G), R6.2
- new net: BZ1.2 (+), Q1.3 (D)
- no-connect marks 13 -> 16
Other:
- note added: "AUX"
- note added: "STEP UP MT3608"
- company: (none) -> E.E.S.T. N°5
- title: (none) -> Alarma_Wifi_ESP8266
- moved on the sheet: C1, C2, C3, C4, C5, D1, D2, J1, J2, J3, R1, R2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

Commit message: Actualizacion PCB
Parts:
- removed U1: TP4056, SOP127P600X175-9N, symbol TP4056_2:TP4056
- added U5: TP4056, TP4056:SOP127P600X175-9N, symbol TP4056:TP4056
- R9: footprint (none) -> Resistor_SMD:R_0805_2012Metric_Pad1.20x1.40mm_HandSolder
- RV1: footprint Potentiometer_THT:Potentiometer_Vishay_T73YP_Vertical -> Potentiometer_THT:Potentiometer_Bourns_3266P_Horizontal
- SW1: footprint (none) -> EESTN5-v2:SW_SPDT_TH_100Mils_VERTICAL
Connections:
- net EP: now also U5.9 (EP)
- net GND: now also U5.1 (TEMP), U5.3 (GND)
- net VB: now also U5.5 (BAT)
- net at C1.2, D1.2 (A), D2.2 (A)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: now also U5.4 (VCC), U5.8 (CE)
- net at R3.1: now also U5.6 (~{STDBY})
- net at R2.1: now also U5.7 (~{CHRG})
- net at R1.2: now also U5.2 (PROG)
Changed lines of the file:
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@@
       (effects (font (size 1.27 1.27)) (justify right))
     )
-    (property "Footprint" "Potentiometer_THT:Potentiometer_Vishay_T73YP_Vertical" (at 78.232 136.144 0)
+    (property "Footprint" "Potentiometer_THT:Potentiometer_Bourns_3266P_Horizontal" (at 78.232 136.144 0)
       (effects (font (size 1.27 1.27)) hide)
     )
@@
       (effects (font (size 1.27 1.27)))
     )
-    (property "Footprint" "" (at 42.418 129.794 0)
+    (property "Footprint" "EESTN5-v2:SW_SPDT_TH_100Mils_VERTICAL" (at 42.418 129.794 0)
       (effects (font (size 1.27 1.27)) hide)
     )
@@
       (effects (font (size 1.27 1.27)) (justify left))
     )
-    (property "Footprint" "" (at 76.454 145.542 90)
+    (property "Footprint" "Resistor_SMD:R_0805_2012Metric_Pad1.20x1.40mm_HandSolder" (at 76.454 145.542 90)
       (effects (font (size 1.27 1.27)) hide)
     )
@@
         (path "/600f7fd8-1170-442d-b793-e33d87c66e69"
           (reference "J2") (unit 1)
+        )
+      )
+    )
+  )
+  (symbol (lib_id "TP4056:TP4056") (at 87.122 63.754 0) (unit 1)
+    (in_bom yes) (on_board yes) (dnp no) (fields_autoplaced)
+    (property "Reference" "U5" (at 87.122 46.736 0)
+      (effects (font (size 1.27 1.27)))
+    )
+    (property "Value" "TP4056" (at 87.122 49.276 0)
+      (effects (font (size 1.27 1.27)))
+    )
+    (property "Footprint" "TP4056:SOP127P600X175-9N" (at 87.122 63.754 0)
+      (effects (font (size 1.27 1.27)) (justify bottom) hide)
+    )
+    (property "Datasheet" "" (at 87.122 63.754 0)
+      (effects (font (size 1.27 1.27)) hide)
+    )
+    (property "STANDARD" "IPC 7351B" (at 87.122 63.754 0)
+      (effects (font (size 1.27 1.27)) (justify bottom) hide)
+    )
+    (property "MAXIMUM_PACKAGE_HEIGHT" "1.75mm" (at 87.122 63.754 0)
+      (effects (font (size 1.27 1.27)) (justify bottom) hide)
+    )
+    (property "MANUFACTURER" "NanJing Top Power ASIC Corp." (at 87.122 63.754 0)
+      (effects (font (size 1.27 1.27)) (justify bottom) hide)
+    )
+    (pin "1")
+    (pin "2")
+    (pin "3")
+    (pin "4")
+    (pin "5")
+    (pin "6")
+    (pin "7")
+    (pin "8")
+    (pin "9")
+    (instances
+      (project "MainBoard_ESP8266"
+        (path "/600f7fd8-1170-442d-b793-e33d87c66e69"
+          (reference "U5") (unit 1)
         )
       )
@@
         )
       )
-    )
-  )
-  (symbol (lib_id "TP4056_2:TP4056") (at 87.122 63.754 0) (unit 1)
-    (in_bom yes) (on_board yes) (dnp no) (fields_autoplaced)
-    (property "Reference" "U1" (at 87.122 46.736 0)
-      (effects (font (size 1.27 1.27)))
-    )
-    (property "Value" "TP4056" (at 87.122 49.276 0)
-      (effects (font (size 1.27 1.27)))
-    )
-    (property "Footprint" "SOP127P600X175-9N" (at 87.122 63.754 0)
-      (effects (font (size 1.27 1.27)) (justify bottom) hide)
-    )
-    (property "Datasheet" "" (at 87.122 63.754 0)
-      (effects (font (size 1.27 1.27)) hide)
-    )
-    (property "STANDARD" "IPC 7351B" (at 87.122 63.754 0)
-      (effects (font (size 1.27 1.27)) (justify bottom) hide)
-    )
-    (property "MAXIMUM_PACKAGE_HEIGHT" "1.75mm" (at 87.122 63.754 0)
-      (effects (font (size 1.27 1.27)) (justify bottom) hide)
-    )
-    (property "MANUFACTURER" "NanJing Top Power ASIC Corp." (at 87.122 63.754 0)
-      (effects (font (size 1.27 1.27)) (justify bottom) hide)
-    )
-    (pin "1")
-    (pin "2")
-    (pin "3")
-    (pin "4")
-    (pin "5")
-    (pin "6")
-    (pin "7")
-    (pin "8")
-    (pin "9")
-    (instances
-      (project "SmartWatch"
-        (path "/33c9733c-ce67-4179-8c61-800eba0b21c9"
-          (reference "U1") (unit 1)
-        )
-      )
-      (project "MainBoard_ESP8266"
-        (path "/600f7fd8-1170-442d-b793-e33d87c66e69"
-          (reference "U1") (unit 1)
-        )
-      )

Commit message: Edicion archivos pcb
Parts:
- removed J3: FTDI, Connector_PinHeader_2.54mm:PinHeader_1x04_P2.54mm_Horizontal, symbol Connector:Conn_01x04_Pin
- added J4: Sensor, Connector_PinHeader_2.54mm:PinHeader_1x03_P2.54mm_Horizontal, symbol Connector:Conn_01x03_Socket
- added J5: FTDI, Connector_PinHeader_2.54mm:PinHeader_1x03_P2.54mm_Horizontal, symbol Connector:Conn_01x03_Socket
Connections:
- net +5V: now also J4.1 (Pin_1)
- net BUZZER: now also U3.7 (GPIO13); no longer U3.5 (GPIO14)
- net GND: now also J4.3 (Pin_3), J5.3 (Pin_3)
- net LED_WIFI: now also U3.5 (GPIO14); no longer U3.7 (GPIO13)
- net Rx: now also J5.2 (Pin_2)
- net Tx: now also J5.1 (Pin_1)
- net PIR: now reaches U3.19 (GPIO4)
- net PIR: now also J4.2 (Pin_2)
- no-connect marks 16 -> 15
Other:
- moved on the sheet: BZ1, D4, D5, Q1, R6

Commit message: Mejoras PCB
Parts:
- added H1: Hole, EESTN5-v2:Separador_M3_5mm, symbol Mechanical:MountingHole
Changed lines of the file:
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@@
+    )
+  )
+  (symbol (lib_id "Mechanical:MountingHole") (at 256.54 126.492 0) (unit 1)
+    (in_bom yes) (on_board yes) (dnp no)
+    (property "Reference" "H1" (at 254.762 121.412 0)
+      (effects (font (size 1.27 1.27)) (justify left))
+    )
+    (property "Value" "Hole" (at 254.762 123.444 0)
+      (effects (font (size 1.27 1.27)) (justify left))
+    )
+    (property "Footprint" "EESTN5-v2:Separador_M3_5mm" (at 256.54 126.492 0)
+      (effects (font (size 1.27 1.27)) hide)
+    )
+    (property "Datasheet" "~" (at 256.54 126.492 0)
+      (effects (font (size 1.27 1.27)) hide)
+    )
+    (instances
+      (project "MainBoard_ESP8266"
+        (path "/600f7fd8-1170-442d-b793-e33d87c66e69"
+          (reference "H1") (unit 1)
+        )
+      )
     )
   )
